File: clock_and_power.kicad_sch (KiCad schematic)
At the start: 16 parts, among them Q1 2N7000, U13 74LS32, U14 NE555P, U15 NE555P, U16 74HC74

Commit message: New pdt plotted
Other:
- title: Scoreboard -> DIGITAL SCOREBOARD
Changed lines of the file:
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@@
   (paper "A4")
   (title_block
-    (title "Scoreboard")
+    (title "DIGITAL SCOREBOARD")
     (rev "1.0")
     (company "www.slemanz.com")
