File: timer.kicad_sch (KiCad schematic)
At the start: 27 parts, among them U17 74LS08, U18 4511, U19 4511, U20 74LS32, U21 4029, U22 4029, U23 4511, U24 4511, U25 4029, U26 4029, U27 74LS04

Commit message: New pdt plotted
Other:
- title: Scoreboard -> DIGITAL SCOREBOARD
Changed lines of the file:
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@@
   (paper "A3")
   (title_block
-    (title "Scoreboard")
+    (title "DIGITAL SCOREBOARD")
     (rev "1.0")
     (company "www.slemanz.com")
