File: Digital_Scoreboard.kicad_sch (KiCad schematic)
At the start: 28 parts, among them SW1 SW_Push, SW2 SW_Push, SW3 SW_Push, SW4 SW_Push, SW5 SW_Push, SW6 SW_Push, U1 D168K, U10 D168K, U11 D168K, U12 D168K, U2 D168K, U3 D168K, U4 D168K, U5 D168K, U6 D168K, U7 D168K, U8 D168K, U9 D168K

Commit message: New pdt plotted
Other:
- title: Scoreboard -> DIGITAL SCOREBOARD
Changed lines of the file:
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@@
   (paper "A3")
   (title_block
-    (title "Scoreboard")
+    (title "DIGITAL SCOREBOARD")
     (rev "1.0")
     (company "www.slemanz.com")

Commit message: error fixed
Other:
- note added: "CLOCK"
- note added: "POWER SUPPLY"
- note added: "UP/DOWN"
- note removed: "CLOCK AND POWER SUPPLY"
- title: DIGITAL SCOREBOARD -> Scoreboard
Changed lines of the file:
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@@
   (paper "A3")
   (title_block
-    (title "DIGITAL SCOREBOARD")
+    (title "Scoreboard")
     (rev "1.0")
     (company "www.slemanz.com")
@@
     )
   )
-  (text "4" (at 43.18 73.66 0)
+  (text "3" (at 62.23 274.32 0)
     (effects (font (size 4 4) (thickness 3) bold (color 132 0 0 1)) (justify right bottom))
   )
-  (text "3" (at 43.18 66.04 0)
+  (text "4" (at 43.18 81.28 0)
+    (effects (font (size 4 4) (thickness 3) bold (color 132 0 0 1)) (justify right bottom))
+  )
+  (text "3" (at 43.18 73.66 0)
+    (effects (font (size 4 4) (thickness 3) bold (color 132 0 0 1)) (justify right bottom))
+  )
+  (text "2" (at 62.23 238.76 0)
+    (effects (font (size 4 4) (thickness 3) bold (color 132 0 0 1)) (justify right bottom))
+  )
+  (text "2" (at 43.18 66.04 0)
     (effects (font (size 4 4) (thickness 3) bold (color 132 0 0 1)) (justify right bottom))
   )
@@
     (effects (font (size 4 4) (thickness 3) bold (color 132 0 0 1)) (justify left bottom))
   )
-  (text "SCORE" (at 53.34 73.66 0)
+  (text "SCORE" (at 53.34 81.28 0)
     (effects (font (size 4 4) (thickness 3) bold (color 132 0 0 1)) (justify left bottom))
   )
+  (text "4" (at 105.41 274.32 0)
+    (effects (font (size 4 4) (thickness 3) bold (color 132 0 0 1)) (justify right bottom))
+  )
   (text "INDEX" (at 53.34 43.18 0)
     (effects (font (size 4 4) (thickness 3) bold (color 0 0 194 1)) (justify left bottom))
   )
-  (text "TIMER" (at 53.34 66.04 0)
+  (text "TIMER" (at 53.34 73.66 0)
     (effects (font (size 4 4) (thickness 3) bold (color 132 0 0 1)) (justify left bottom))
   )
@@
     (effects (font (size 4 4) (thickness 3) bold (color 132 0 0 1)) (justify right bottom))
   )
+  (text "UP/DOWN" (at 306.07 151.13 0)
+    (effects (font (size 3 3) (thickness 3) bold (color 72 0 0 1)) (justify left bottom))
+  )
   (text "DIGITAL SCOREBOARD" (at 139.7 40.005 0)
     (effects (font (size 10 10) (thickness 3) bold (color 132 0 0 1)) (justify left bottom))
@@
     (effects (font (size 7 7) (thickness 3) bold (color 132 0 0 1)) (justify left bottom))
   )
-  (text "CLOCK AND POWER SUPPLY" (at 53.34 58.42 0)
+  (text "CLOCK" (at 53.34 58.42 0)
     (effects (font (size 4 4) (thickness 3) bold (color 132 0 0 1)) (justify left bottom))
   )
@@
     (effects (font (size 6 6) (thickness 3) bold (color 72 0 0 1)) (justify left bottom))
   )
+  (text "POWER SUPPLY" (at 53.34 66.04 0)
+    (effects (font (size 4 4) (thickness 3) bold (color 132 0 0 1)) (justify left bottom))
+  )
   (global_label "T_QE_3" (shape input) (at 155.575 93.98 180) (fields_autoplaced)
