File: score.kicad_sch (KiCad schematic)
At the start: 40 parts, among them U42 74LS32, U43 74LS08, U44 74LS04

Commit message: New pdt plotted
Other:
- title: Scoreboard -> DIGITAL SCOREBOARD
Changed lines of the file:
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@@
   (paper "A3")
   (title_block
-    (title "Scoreboard")
+    (title "DIGITAL SCOREBOARD")
     (rev "1.0")
     (company "www.slemanz.com")

Commit message: error fixed 2
Other:
- note added: "[04] SCORE"
- note removed: "[03] SCORE"
Changed lines of the file:
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@@
     (effects (font (size 1.27 1.27) (thickness 0.254) bold (color 132 0 0 1)) (justify left top))
   )
-  (text "[03] SCORE" (at 177.165 27.94 0)
+  (text "[04] SCORE" (at 177.165 27.94 0)
     (effects (font (size 8 8) (thickness 0.8) bold (color 132 0 0 1)) (justify left bottom))
   )
